Commit message: Robot Model Added

File: description/robot_core.xacro (robot description, xacro)
@@ -27,6 +27,6 @@
     </joint>
     <link name="chassis">
-        <xacro:insert_box_with_fillet size_x="0.28" size_y="0.2" size_z="${chassis_height}"
-        fillet_radius="0.02" material="orange" x="0.09" y="0" z="${chassis_height/2}"/>
+        <!-- <xacro:insert_box_with_fillet size_x="0.28" size_y="0.2" size_z="${chassis_height}"
+        fillet_radius="0.02" material="silver" x="0.09" y="0" z="${chassis_height/2}"/>
         <collision>
            <origin xyz="0.09 0 ${chassis_height/2}" rpy="0 0 0"/>
@@ -34,7 +34,8 @@
                 <box size="0.28 0.2 ${chassis_height}"/>
             </geometry>
-        </collision>
+        </collision> -->
+        <!-- Chassis Main Body -->
         <xacro:insert_box_with_fillet size_x="0.4" size_y="0.1" size_z="${chassis_height}"
-        fillet_radius="0.02" material="orange" x="0.15" y="0" z="${chassis_height/2}"/>
+        fillet_radius="0.02" material="silver" x="0.15" y="0" z="${chassis_height/2}"/>
         <collision>
            <origin xyz="0.15 0 ${chassis_height/2}" rpy="0 0 0"/>
@@ -43,4 +44,5 @@
             </geometry>
         </collision>
+        <!-- Chassis Cylinder Rod -->
         <visual>
             <origin xyz="0 0 0" rpy="${-pi/2} 0 0"/>
@@ -72,5 +74,6 @@
     </link>
     <gazebo reference="chassis">
-        <material>Gazebo/Orange</material>
+        <material>Gazebo/<color rgba="1.0 0.0 0.0 0.0"/>
+        </material>
     </gazebo>
     <!--  ########################### -->
