Commit message: Added camera

File: description/robot.urdf.xacro (robot description, xacro)
@@ -1,4 +1,8 @@
 <?xml version="1.0"?>
 <robot xmlns:xacro="http://www.ros.org/wiki/xacro" name="traktor">
+    <xacro:include filename="sensors/sonar.xacro"/>
+    <xacro:include filename="sensors/lidar.xacro"/>
+    <!-- <xacro:include filename="sensors/imu.xacro"/> -->
+    <!-- <xacro:include filename="sensors/cam.xacro"/> -->
 <link name="base_link">
   <inertial>
@@ -363,9 +367,9 @@
   </gazebo>
 <!-- LİDAR LİNK -->
-  <link name="hokuyo_link">
+  <link name="lidar_link">
     <collision>
       <origin xyz="0 0 0" rpy="0 0 0"/>
       <geometry>
-        <cylinder radius="0.05" length="0.05"/>
+        <cylinder radius="0.1" length="0.1"/>
       </geometry>
     </collision>
@@ -373,5 +377,5 @@
       <origin xyz="0 0 0" rpy="0 0 0"/>
       <geometry>
-        <cylinder radius="0.05" length="0.05"/>
+        <cylinder radius="0.1" length="0.1"/>
       </geometry>
     </visual>
@@ -382,17 +386,17 @@
     </inertial>
   </link>
-  <joint name="hokuyo_joint" type="fixed">
+  <joint name="lidar_joint" type="fixed">
     <axis xyz="0 1 0" />
     <origin xyz="1 0 0.51" rpy="0 0 0"/>
     <parent link="base_link"/>
-    <child link="hokuyo_link"/>
+    <child link="lidar_link"/>
   </joint>
 <!-- LİDAR PLUGİN -->
-<gazebo reference="hokuyo_link">
-    <sensor name="hokuyo_link" type="ray">
+<gazebo reference="lidar_link">
+    <sensor name="lidar" type="ray">
       <pose>0.215 0 0.215 0 0 0</pose>
       <always_on>true</always_on>
       <visualize>true</visualize>
-      <update_rate>5</update_rate>
+      <update_rate>10</update_rate>
       <ray>
         <scan>
@@ -400,11 +404,11 @@
             <samples>360</samples>
             <resolution>1.00000</resolution>
-            <min_angle>0.000000</min_angle>
-            <max_angle>6.280000</max_angle>
+            <min_angle>-3.14</min_angle>
+            <max_angle>3.14</max_angle>
           </horizontal>
         </scan>
         <range>
           <min>0.120000</min>
-          <max>3.5</max>
+          <max>15</max>
           <resolution>0.015000</resolution>
         </range>
@@ -425,4 +429,92 @@
     <material>Gazebo/Red</material>
   </gazebo>
+  <!-- Camera link -->
+    <joint name="cam_joint" type="fixed">
+        <parent link="base_link"/>
+        <child link="cam_link"/>
+        <origin xyz="1.25 0 0.41" rpy="0 0 0"/>
+    </joint>
+    <link name="cam_link">
+        <visual>
+            <geometry>
+                <box size="0.030 0.05 0.05"/>
+            </geometry>
+            <material name="black"/>
+        </visual>
+    </link>
+    <joint name="cam_optical_joint" type="fixed">
+        <parent link="cam_link"/>
+        <child link="cam_link_optical"/>
+        <origin xyz="0 0 0" rpy="${-pi/2} 0 ${-pi/2}"/>
+    </joint>
+    <link name="cam_link_optical"> </link>
+    <gazebo reference="cam_link">
+        <material>Gazebo/Turquoise</material>
+        <sensor name="camera" type="camera">
+            <pose> 0 0 0 0 0 0 </pose>
+            <visualize>true</visualize>
+            <update_rate>10</update_rate>
+            <camera>
+                <horizontal_fov>1.089</horizontal_fov>
+                <image>
+                    <format>R8G8B8</format>
+                    <width>640</width>
+                    <height>480</height>
+                </image>
+                <clip>
+                    <near>0.05</near>
+                    <far>8.0</far>
+                </clip>
+            </camera>
+            <plugin name="camera_controller" filename="libgazebo_ros_camera.so">
+                <frame_name>cam_link_optical</frame_name>
+            </plugin>
+        </sensor>
+    </gazebo>
+  <!--Depth camera link -->
+    <joint name="depth_cam_joint" type="fixed">
+        <parent link="base_link"/>
+        <child link="depth_cam_link"/>
+        <origin xyz="1.25 0 0.48" rpy="0 0 0"/>
+    </joint>
+    <link name="depth_cam_link">
+        <visual>
+            <geometry>
+                <box size="0.030 0.1 0.05"/>
+            </geometry>
+            <material name="black"/>
+        </visual>
+    </link>
+    <joint name="depth_cam_optical_joint" type="fixed">
+        <parent link="depth_cam_link"/>
+        <child link="depth_cam_link_optical"/>
+        <origin xyz="0 0 0" rpy="${-pi/2} 0 ${-pi/2}"/>
+    </joint>
+    <link name="depth_cam_link_optical"> </link>
+    <gazebo reference="depth_cam_link">
+        <material>Gazebo/Turquoise</material>
+        <sensor name="depth_camera" type="depth">
+            <pose> 0 0 0 0 0 0 </pose>
+            <visualize>true</visualize>
+            <update_rate>10</update_rate>
+            <camera>
+                <horizontal_fov>1.089</horizontal_fov>
+                <image>
+                    <format>B8R8G8</format>
+                    <width>640</width>
+                    <height>480</height>
+                </image>
+                <clip>
+                    <near>0.05</near>
+                    <far>8.0</far>
+                </clip>
+            </camera>
+            <plugin name="depth_camera_controller" filename="libgazebo_ros_camera.so">
+                <frame_name>depth_cam_link_optical</frame_name>
+                <min_depth>0.1</min_depth>
+                <max_depth>100</max_depth>
+            </plugin>
+        </sensor>
+    </gazebo>
 <!-- ACKERMANN DRİVE PLUGİN  -->
 <gazebo>

File: description/sensors/cam.xacro (robot description, xacro)
@@ -1,74 +1,31 @@
 <?xml version="1.0"?>
 <robot xmlns:xacro="http://www.ros.org/wiki/xacro" >
-    <xacro:macro name="insert_camera" params="base_name parent_name x y z mass width height min_range max_range tilt_angle visualize">
-        <joint name="${base_name}_joint" type="fixed">
-            <parent link="${parent_name}"/>
-            <child link="${base_name}"/>
-            <origin xyz="${x} ${y} ${z}" rpy="0 ${tilt_angle} 0"/>
-        </joint>
-        <link name="${base_name}">
-            <visual>
-                <origin xyz="-0.02 0 0" rpy="0 ${-pi/2} 0"/>
-                <geometry>
-                    <cylinder radius="0.015" length="0.04"/>
-                </geometry>
-                <material name="grey"/>
-            </visual>
-            <visual>
-                <origin xyz="-0.03 0 0" rpy="0 ${-pi/2} 0"/>
-                <geometry>
-                    <!-- <cylinder radius="0.03" length="0.02"/> -->
-                    <box size="0.04 0.06 0.02"/>
-                </geometry>
-                <material name="grey"/>
-            </visual>
-            <collision>
-                <origin xyz="-0.02 0 0" rpy="0 ${-pi/2} 0"/>
-                <geometry>
-                    <cylinder radius="0.02" length="0.04"/>
-                </geometry>
-            </collision>
-            <xacro:inertial_cylinder mass="${mass}" radius="0.02" length="0.04">
-                <origin xyz="-0.02 0 0" rpy="0 ${-pi/2} 0"/>
-            </xacro:inertial_cylinder>
-        </link>
-        <joint name="${base_name}_optical_joint" type="fixed">
-            <parent link="${base_name}"/>
-            <child link="${base_name}_optical_link"/>
-            <origin xyz="0 0 0" rpy="${-pi/2} 0 ${-pi/2}"/>
-        </joint>
-        <link name="${base_name}_optical_link"/>
-        <gazebo reference="${base_name}">
-          <material>Gazebo/DarkGrey</material>
-          <sensor name="${base_name}" type="camera">
-            <pose> 0 0 0 0 0 0 </pose>
-            <visualize>${visualize}</visualize>
-            <update_rate>20</update_rate>
-            <camera>
-                <!-- <horizontal_fov>1.089</horizontal_fov> -->
-                <horizontal_fov>1.46608</horizontal_fov>
-                <image>
-                    <format>R8G8B8</format>
-                    <width>${width}</width>
-                    <height>${height}</height>
-                </image>
-                <clip>
-                    <near>${min_range}</near>
-                    <far>${max_range}</far>
-                </clip>
-            </camera>
-            <plugin name="${base_name}_plugin" filename="libgazebo_ros_camera.so">
-                <frame_name>${base_name}_optical_link</frame_name>
-            </plugin>
-          </sensor>
-        </gazebo>
-    </xacro:macro>
-</robot>
- <!-- <joint name="line_cam_joint" type="fixed">
-        <parent link="chassis"/>
+    <gazebo reference="cam_link">
+        <material>Gazebo/Red</material>
+    </gazebo>
+    <gazebo reference="right_wheel_steer">
+        <material>Gazebo/Green</material>
+    </gazebo>
+    <gazebo reference="left_wheel_steer">
+        <material>Gazebo/Green</material>
+    </gazebo>
+    <gazebo reference="front_right_wheel">
+        <material>Gazebo/Black</material>
+    </gazebo>
+    <gazebo reference="front_left_wheel">
+        <material>Gazebo/Black</material>
+    </gazebo>
+    <gazebo reference="rear_left_wheel">
+        <material>Gazebo/Black</material>
+    </gazebo>
+    <gazebo reference="rear_right_wheel">
+        <material>Gazebo/Black</material>
+    </gazebo>
+    <joint name="cam_joint" type="fixed">
+        <parent link="base_link"/>
         <child link="line_cam"/>
-        <origin xyz="0.305 0 0.08" rpy="0 0 0"/>
+        <origin xyz="2.5 0 0.51" rpy="0 0 0"/>
     </joint>
-    <link name="line_cam">
+    <link name="cam_link">
         <visual>
             <geometry>
@@ -78,13 +35,13 @@
         </visual>
     </link>
-    <joint name="line_cam_optical_joint" type="fixed">
-        <parent link="line_cam"/>
-        <child link="line_cam_link_optical"/>
+    <joint name="cam_optical_joint" type="fixed">
+        <parent link="cam_link"/>
+        <child link="cam_link_optical"/>
         <origin xyz="0 0 0" rpy="${-pi/2} 0 ${-pi/2}"/>
     </joint>
-    <link name="line_cam_link_optical"></link>
-    <gazebo reference="line_cam">
+    <link name="cam_link_optical"> </link>
+    <gazebo reference="cam_link">
         <material>Gazebo/Red</material>
-        <sensor name="line_cam" type="camera">
+        <!-- <sensor name="line_cam" type="camera">
             <pose> 0 0 0 0 0 0 </pose>
             <visualize>true</visualize>
@@ -105,4 +62,5 @@
                 <frame_name>line_cam_link_optical</frame_name>
             </plugin>
-        </sensor>
-    </gazebo> -->
+        </sensor> -->
+    </gazebo>
+</robot>

Commit message: ros2_control remove

File: description/robot.urdf.xacro (robot description, xacro)
@@ -1,8 +1,9 @@
 <?xml version="1.0"?>
 <robot xmlns:xacro="http://www.ros.org/wiki/xacro" name="traktor">
-    <xacro:include filename="sensors/sonar.xacro"/>
-    <xacro:include filename="sensors/lidar.xacro"/>
+    <!-- <xacro:include filename="sensors/sonar.xacro"/> -->
+    <!-- <xacro:include filename="sensors/lidar.xacro"/> -->
     <!-- <xacro:include filename="sensors/imu.xacro"/> -->
     <!-- <xacro:include filename="sensors/cam.xacro"/> -->
+    <xacro:include filename="ros2_control.xacro"/>
 <link name="base_link">
   <inertial>
@@ -210,5 +211,5 @@
   </collision>
 </link>
-<joint name="rear_left_wheel_joint" type="continuous"> <!-- SOL ARKA TEKER DİFERANSİYEL VE SOL ARKA TEKER JOİNTİ-->
+<joint name="rear_left_wheel_joint" type="continuous">
   <parent link="base_link"/>
   <child link="rear_left_wheel"/>
