Commit message: added ackermann plugin

File: description/controllers/gazebo_hw_ros2_control.xacro (robot description, xacro)
@@ -2,23 +2,4 @@
 <robot xmlns:xacro="http://ros.org/wiki/xacro">
     <xacro:include filename="transmission_macros.xacro"/>
-    <ros2_control name="GazeboSystem" type="system">
-        <hardware>
-            <plugin>gazebo_ros2_control/GazeboSystem</plugin>
-        </hardware>
-        <xacro:insert_servo_transmission joint_name="front_left_servo_joint"/>
-        <xacro:insert_servo_transmission joint_name="front_right_servo_joint"/>
-        <xacro:insert_wheel_transmission joint_name="front_left_wheel_joint"/>
-        <xacro:insert_wheel_transmission joint_name="front_right_wheel_joint"/>
-        <xacro:insert_wheel_transmission joint_name="rear_left_wheel_joint"/>
-        <xacro:insert_wheel_transmission joint_name="rear_right_wheel_joint"/>
-    </ros2_control>
-    <gazebo>
-        <plugin filename="libgazebo_ros2_control.so" name="gazebo_ros2_control">
-            <robot_param>robot_description</robot_param>
-            <robot_namespace>ebot</robot_namespace>
-            <robot_param_node>robot_state_publisher</robot_param_node>
-            <parameters>$(find ebot)/config/robo_car_controllers.yaml</parameters>
-        </plugin>
-    </gazebo>
     <gazebo>
         <plugin name="joint_state" filename="libgazebo_ros_joint_state_publisher.so">
@@ -35,3 +16,45 @@
         </plugin>
     </gazebo>
+    <gazebo>
+        <plugin name="gazebo_ros_ackermann_drive" filename="libgazebo_ros_ackermann_drive.so">
+            <ros>
+                <namespace>demo</namespace>
+                <remapping>cmd_vel:=cmd_demo</remapping>
+                <remapping>odom:=odom_demo</remapping>
+                <remapping>distance:=distance_demo</remapping>
+                <remapping>steerangle:=steerangle_demo</remapping>
+            </ros>
+            <update_rate>30.0</update_rate>
+            <!-- wheels -->
+            <front_left_joint>front_left_wheel_joint</front_left_joint>
+            <front_right_joint>front_right_wheel_joint</front_right_joint>
+            <rear_left_joint>rear_left_wheel_joint</rear_left_joint>
+            <rear_right_joint>rear_right_wheel_joint</rear_right_joint>
+            <left_steering_joint>front_left_servo_joint</left_steering_joint>
+            <right_steering_joint>front_right_servo_joint</right_steering_joint>
+            <steering_wheel_joint>steering_joint</steering_wheel_joint>
+            <!-- Max absolute steer angle for tyre in radians-->
+            <!-- Any cmd_vel angular z greater than this would be capped -->
+            <max_steer>0.6458</max_steer>
+            <!-- Max absolute steering angle of steering wheel -->
+            <max_steering_angle>7.85</max_steering_angle>
+            <!-- Max absolute linear speed in m/s -->
+            <max_speed>20</max_speed>
+            <!-- PID tuning -->
+            <left_steering_pid_gain>1500 0 1</left_steering_pid_gain>
+            <left_steering_i_range>0 0</left_steering_i_range>
+            <right_steering_pid_gain>1500 0 1</right_steering_pid_gain>
+            <right_steering_i_range>0 0</right_steering_i_range>
+            <linear_velocity_pid_gain>1000 0 1</linear_velocity_pid_gain>
+            <linear_velocity_i_range>0 0</linear_velocity_i_range>
+            <!-- output -->
+            <publish_odom>true</publish_odom>
+            <publish_odom_tf>true</publish_odom_tf>
+            <publish_wheel_tf>true</publish_wheel_tf>
+            <publish_distance>true</publish_distance>
+            <publish_steerangle>true</publish_steerangle>
+            <odometry_frame>odom_demo</odometry_frame>
+            <robot_base_frame>base_link</robot_base_frame>
+        </plugin>
+    </gazebo>
 </robot>

File: description/robot.urdf.xacro (robot description, xacro)
@@ -1,7 +1,489 @@
 <?xml version="1.0"?>
-<robot name="ebot" xmlns:xacro="http://www.ros.org/wiki/xacro">
-    <xacro:include filename="color_macros.xacro" />
-    <xacro:include filename="inertia_macros.xacro" />
-    <xacro:include filename="robot_core.xacro" />
-    <xacro:include filename="controllers/gazebo_hw_ros2_control.xacro" />
+<robot xmlns:xacro="http://www.ros.org/wiki/xacro" name="traktor">
+<link name="base_link">
+  <inertial>
+    <origin xyz="0.0 0.0 0.0" rpy="0.0 0.0 0.0"/>
+    <mass value="10"/>
+    <inertia ixx="24.166666666666668" ixy="0" ixz="0" iyy="28.333333333333336" iyz="0" izz="10.833333333333334"/>
+  </inertial>
+  <visual name="chassis">
+    <origin xyz="0.0 0.0 0.0" rpy="0.0 0.0 0.0"/>
+    <!--  <mesh filename="package://your_package/meshes/your_mesh.stl"/> -->
+    <geometry>
+      <box size="2.5 1.2 1"/>
+    </geometry>
+    <material name="">
+      <color rgba="1.0 0.0 0.0 1.0"/>
+      <texture filename=""/>
+    </material>
+  </visual>
+  <collision>
+    <origin xyz="0.0 0.0 0.0" rpy="0.0 0.0 0.0"/>
+    <!--  <mesh filename="package://your_package/meshes/your_mesh.stl"/> -->
+    <geometry>
+      <box size="2.5 1.2 1"/>
+    </geometry>
+  </collision>
+</link>
+<!-- Right wheel steer  -->
+<link name="right_wheel_steer">
+  <visual>
+    <geometry>
+      <cylinder length="0.05" radius="0.02"/>
+    </geometry>
+    <material name="black"/>
+  </visual>
+  <collision>
+    <geometry>
+      <cylinder length="0.05" radius="0.02"/>
+    </geometry>
+  </collision>
+  <inertial>
+    <origin xyz="0.0 0.0 0.0" rpy="0.0 0.0 0.0"/>
+    <mass value="1"/>
+    <inertia ixx="0.07583333333333334" ixy="0" ixz="0" iyy="0.07583333333333334" iyz="0" izz="0.125"/>
+  </inertial>
+</link>
+<joint name="right_wheel_steer_joint" type="revolute">
+  <parent link="base_link"/>
+  <child link="right_wheel_steer"/>
+  <origin xyz="0.75 -0.85 -0.5" rpy="1.5707 0 0"/>
+  <axis xyz="0 1 0"/>
+  <limit effort="100" velocity="1" lower="-1" upper="1"/>
+  <dynamics damping="0.0" friction="0.0"/>
+</joint>
+<!-- Front right wheel -->
+<link name="front_right_wheel">
+  <inertial>
+    <origin xyz="0.0 0.0 0.0" rpy="0.0 0.0 0.0"/>
+    <mass value="1"/>
+    <inertia ixx="0.07583333333333334" ixy="0" ixz="0" iyy="0.07583333333333334" iyz="0" izz="0.125"/>
+  </inertial>
+  <visual name="">
+    <origin xyz="0.0 0.0 0.0" rpy="0.0 0.0 0.0"/>
+    <!--  <mesh filename="package://your_package/meshes/your_mesh.stl"/> -->
+    <geometry>
+      <cylinder length="0.20" radius="0.25"/>
+    </geometry>
+    <material name="">
+      <color rgba="0.0 0.0 0.0 1.0"/>
+      <texture filename=""/>
+    </material>
+  </visual>
+  <collision>
+    <origin xyz="0.0 0.0 0.0" rpy="0.0 0.0 0.0"/>
+    <!--  <mesh filename="package://your_package/meshes/your_mesh.stl"/> -->
+    <geometry>
+      <cylinder length="0.20" radius="0.25"/>
+    </geometry>
+  </collision>
+</link>
+<joint name="front_right_wheel_joint" type="continuous">
+  <parent link="right_wheel_steer"/>
+  <child link="front_right_wheel"/>
+  <origin xyz="0.0 0.0 0.0" rpy="0 0 0"/>
+  <axis xyz="0 0 -1"/>
+  <limit effort="100" velocity="100"/>
+  <dynamics damping="0.0" friction="0.0"/>
+</joint>
+<!-- Rear right wheel -->
+<link name="rear_right_wheel">
+  <inertial>
+    <origin xyz="0.0 0.0 0.0" rpy="0.0 0.0 0.0"/>
+    <mass value="1"/>
+    <inertia ixx="0.07583333333333334" ixy="0" ixz="0" iyy="0.07583333333333334" iyz="0" izz="0.125"/>
+  </inertial>
+  <visual name="">
+    <origin xyz="0.0 0.0 0.0" rpy="0.0 0.0 0.0"/>
+    <!--  <mesh filename="package://your_package/meshes/your_mesh.stl"/> -->
+    <geometry>
+      <cylinder length="0.20" radius="0.4"/>
+    </geometry>
+    <material name="">
+      <color rgba="0.0 0.0 0.0 1.0"/>
+      <texture filename=""/>
+    </material>
+  </visual>
+  <collision>
+    <origin xyz="0.0 0.0 0.0" rpy="0.0 0.0 0.0"/>
+    <!--  <mesh filename="package://your_package/meshes/your_mesh.stl"/> -->
+    <geometry>
+      <cylinder length="0.20" radius="0.4"/>
+    </geometry>
+  </collision>
+</link>
+<joint name="rear_right_wheel_joint" type="continuous">
+  <parent link="base_link"/>
+  <child link="rear_right_wheel"/>
+    <origin xyz="-1.25 -0.85 -0.35" rpy="1.5707 0 0"/>
+  <axis xyz="0 0 -1"/>
+  <limit effort="100" velocity="100"/>
+  <dynamics damping="0.0" friction="0.0"/>
+</joint>
+<!-- Left_wheel_steer -->
+<link name="left_wheel_steer">
+  <inertial>
+    <origin xyz="0.0 0.0 0.0" rpy="0.0 0.0 0.0"/>
+    <mass value="1"/>
+    <inertia ixx="0.07583333333333334" ixy="0" ixz="0" iyy="0.07583333333333334" iyz="0" izz="0.125"/>
+  </inertial>
+  <visual>
+    <geometry>
+      <cylinder length="0.05" radius="0.02"/>
+    </geometry>
+    <collision>
+      <geometry>
+        <cylinder length="0.05" radius="0.02"/>
+      </geometry>
+    </collision>
+    <material name="black"/>
+  </visual>
+</link>
+<joint name="left_wheel_steer_joint" type="revolute">
+  <parent link="base_link"/>
+  <child link="left_wheel_steer"/>
+  <origin xyz="0.75 0.85 -0.5" rpy="1.5707 0 0"/>
+  <axis xyz="0 1 0"/>
+  <limit effort="100" velocity="1" lower="-1" upper="1"/>
+  <dynamics damping="0.0" friction="0.0"/>
+</joint>
+<!-- Front left wheel -->
+<link name="front_left_wheel">
+  <inertial>
+    <origin xyz="0.0 0.0 0.0" rpy="0.0 0.0 0.0"/>
+    <mass value="1"/>
+    <inertia ixx="0.07583333333333334" ixy="0" ixz="0" iyy="0.07583333333333334" iyz="0" izz="0.125"/>
+  </inertial>
+  <visual name="">
+    <origin xyz="0.0 0.0 0.0" rpy="0.0 0.0 0.0"/>
+    <!--  <mesh filename="package://your_package/meshes/your_mesh.stl"/> -->
+    <geometry>
+      <cylinder length="0.20" radius="0.25"/>
+    </geometry>
+    <material name="">
+      <color rgba="0.0 0.0 0.0 1.0"/>
+      <texture filename=""/>
+    </material>
+  </visual>
+  <collision>
+    <origin xyz="0.0 0.0 0.0" rpy="0.0 0.0 0.0"/>
+    <!--  <mesh filename="package://your_package/meshes/your_mesh.stl"/> -->
+    <geometry>
+      <cylinder length="0.20" radius="0.25"/>
+    </geometry>
+  </collision>
+</link>
+<joint name="front_left_wheel_joint" type="continuous">
+  <parent link="left_wheel_steer"/>
+  <child link="front_left_wheel"/>
+  <origin xyz="0.0 0.0 0.0" rpy="0 0 0"/>
+  <axis xyz="0 0 -1"/>
+  <limit effort="100" velocity="100"/>
+  <dynamics damping="0.0" friction="0.0"/>
+</joint>
+<!-- Rear left wheel -->
+<link name="rear_left_wheel">
+  <inertial>
+    <origin xyz="0.0 0.0 0.0" rpy="0.0 0.0 0.0"/>
+    <mass value="1"/>
+    <inertia ixx="0.07583333333333334" ixy="0" ixz="0" iyy="0.07583333333333334" iyz="0" izz="0.125"/>
+  </inertial>
+  <visual name="">
+    <origin xyz="0.0 0.0 0.0" rpy="0.0 0.0 0.0"/>
+    <geometry>
+      <cylinder length="0.20" radius="0.4"/>
+    </geometry>
+    <material name="">
+      <color rgba="0.0 0.0 0.0 1.0"/>
+      <texture filename=""/>
+    </material>
+  </visual>
+  <collision>
+    <origin xyz="0.0 0.0 0.0" rpy="0.0 0.0 0.0"/>
+    <geometry>
+      <cylinder length="0.20" radius="0.4"/>
+    </geometry>
+  </collision>
+</link>
+<joint name="rear_left_wheel_joint" type="continuous"> <!-- SOL ARKA TEKER DİFERANSİYEL VE SOL ARKA TEKER JOİNTİ-->
+  <parent link="base_link"/>
+  <child link="rear_left_wheel"/>
+    <origin xyz="-1.25 0.85 -0.35" rpy="1.5707 0 0"/>
+  <axis xyz="0 0 -1"/>
+  <limit effort="100" velocity="100"/>
+  <dynamics damping="0.0" friction="0.0"/>
+</joint>
+<!-- GPS LINK -->
+<link name="gps_link">
+  <inertial>
+    <origin xyz="0.0 0.0 0.0" rpy="0.0 0.0 0.0"/>
+    <mass value="0.1"/>
+    <inertia ixx="0.001" ixy="0" ixz="0" iyy="0.001" iyz="0" izz="0.001"/>
+  </inertial>
+  <visual name="">
+    <origin xyz="0.0 0.0 0.0" rpy="0.0 0.0 0.0"/>
+    <geometry>
+      <box size="0.1 0.1 0.1"/>
+    </geometry>
+    <material name="">
+      <color rgba="0.0 0.0 0.0 1.0"/>
+      <texture filename=""/>
+    </material>
+  </visual>
+  <collision>
+    <origin xyz="0.0 0.0 0.0" rpy="0.0 0.0 0.0"/>
+    <geometry>
+      <box size="0.1 0.1 0.1"/>
+    </geometry>
+  </collision>
+</link>
+<!-- GPS JOINT -->
+<joint name="gps_joint" type="fixed">
+  <parent link="base_link"/>
+  <child link="gps_link"/>
+  <origin xyz="0.0 0.0 0" rpy="0.0 0.0 0.0"/>
+</joint>
+<!-- GPS PLUGIN -->
+  <gazebo reference="gps_link">
+    <sensor name="gps_sensor" type="gps">
+      <always_on>true</always_on>
+      <update_rate>1.0</update_rate>
+      <plugin name="gps_controller" filename="libgazebo_ros_gps_sensor.so">
+        <ros>
+          <!-- <namespace>/br</namespace> -->
+          <remapping>gps_controller/out:=/gps/fix</remapping>
+        </ros>
+        <frame_name>gps_link</frame_name>
+        <offset>0 0 0</offset>
+        <drift>0.001 0.001 0.001</drift>
+        <gaussianNoise>0.05 0.05 0.05</gaussianNoise>
+        <velocityDrift>0.001 0.001 0.001</velocityDrift>
+        <velocityGaussianNoise>0.5 0.5 0.5</velocityGaussianNoise>
+      </plugin>
+    </sensor>
+    <material>Gazebo/Turquoise</material>
+  </gazebo>
+<!-- İMU SENSÖR LİNK,JOİNT -->
+<link name="imu_link">
+  <inertial>
+    <origin xyz="0.0 0.0 0.0" rpy="0.0 0.0 0.0"/>
+    <mass value="0.01"/>
+    <inertia ixx="0.0001" ixy="0.0" ixz="0.0" iyy="0.0001" iyz="0.0" izz="0.0001"/>
+  </inertial>
+  <visual name="">
+    <origin xyz="0.0 0.0 0.0" rpy="0.0 0.0 0.0"/>
+    <geometry>
+      <box size="0.1 0.1 0.02"/>
+    </geometry>
+    <material name="">
+      <color rgba="1.0 0.0 0.0 1.0"/>
+      <texture filename=""/>
+    </material>
+  </visual>
+  <collision>
+    <origin xyz="0.0 0.0 0.0" rpy="0.0 0.0 0.0"/>
+    <geometry>
+      <box size="0.1 0.1 0.02"/>
+    </geometry>
+  </collision>
+</link>
+<joint name="imu_joint" type="fixed">
+  <parent link="base_link"/>
+  <child link="imu_link"/>
+  <origin xyz="1.0 0.0 0" rpy="0.0 0.0 0.0"/>
+</joint>
+<!-- İMU SENSÖR PLUGİN -->
+  <gazebo reference="imu_link">
+    <sensor name="imu_sensor" type="imu">
+      <plugin filename="libgazebo_ros_imu_sensor.so" name="imu_plugin">
+        <ros>
+          <remapping>~/out:=/imu</remapping>
+        </ros>
+        <initial_orientation_as_reference>false</initial_orientation_as_reference>
+      </plugin>
+      <always_on>true</always_on>
+      <update_rate>100</update_rate>
+      <visualize>true</visualize>
+      <imu>
+        <angular_velocity>
+          <x>
+            <noise type="gaussian">
+              <mean>0.0</mean>
+              <stddev>2e-4</stddev>
+              <bias_mean>0.0000075</bias_mean>
+              <bias_stddev>0.0000008</bias_stddev>
+            </noise>
+          </x>
+          <y>
+            <noise type="gaussian">
+              <mean>0.0</mean>
+              <stddev>2e-4</stddev>
+              <bias_mean>0.0000075</bias_mean>
+              <bias_stddev>0.0000008</bias_stddev>
+            </noise>
+          </y>
+          <z>
+            <noise type="gaussian">
+              <mean>0.0</mean>
+              <stddev>2e-4</stddev>
+              <bias_mean>0.0000075</bias_mean>
+              <bias_stddev>0.0000008</bias_stddev>
+            </noise>
+          </z>
+        </angular_velocity>
+        <linear_acceleration>
+          <x>
+            <noise type="gaussian">
+              <mean>0.0</mean>
+              <stddev>1.7e-2</stddev>
+              <bias_mean>0.1</bias_mean>
+              <bias_stddev>0.001</bias_stddev>
+            </noise>
+          </x>
+          <y>
+            <noise type="gaussian">
+              <mean>0.0</mean>
+              <stddev>1.7e-2</stddev>
+              <bias_mean>0.1</bias_mean>
+              <bias_stddev>0.001</bias_stddev>
+            </noise>
+          </y>
+          <z>
+            <noise type="gaussian">
+              <mean>0.0</mean>
+              <stddev>1.7e-2</stddev>
+              <bias_mean>0.1</bias_mean>
+              <bias_stddev>0.001</bias_stddev>
+            </noise>
+          </z>
+        </linear_acceleration>
+      </imu>
+    </sensor>
+    <material>Gazebo/Turquoise</material>
+  </gazebo>
+<!-- LİDAR LİNK -->
+  <link name="hokuyo_link">
+    <collision>
+      <origin xyz="0 0 0" rpy="0 0 0"/>
+      <geometry>
+        <cylinder radius="0.05" length="0.05"/>
+      </geometry>
+    </collision>
+    <visual>
+      <origin xyz="0 0 0" rpy="0 0 0"/>
+      <geometry>
+        <cylinder radius="0.05" length="0.05"/>
+      </geometry>
+    </visual>
+    <inertial>
+      <mass value="1e-5" />
+      <origin xyz="0 0 0" rpy="0 0 0"/>
+      <inertia ixx="1e-6" ixy="0" ixz="0" iyy="1e-6" iyz="0" izz="1e-6" />
+    </inertial>
+  </link>
+  <joint name="hokuyo_joint" type="fixed">
+    <axis xyz="0 1 0" />
+    <origin xyz="1 0 0.51" rpy="0 0 0"/>
+    <parent link="base_link"/>
+    <child link="hokuyo_link"/>
+  </joint>
+<!-- LİDAR PLUGİN -->
+<gazebo reference="hokuyo_link">
+    <sensor name="hokuyo_link" type="ray">
+      <pose>0.215 0 0.215 0 0 0</pose>
+      <always_on>true</always_on>
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
File: description/robot_core.xacro (robot description, xacro)
@@ -17,14 +17,14 @@
     <!-- BASE LINK -->
     <!-- <base joint/> -->
-    <link name="base_link">
-    </link>
+    <!-- <link name="base_link">
+    </link> -->
     <!-- ################# -->
     <!-- CHASSIS LINK -->
-    <joint name="chassis_joint" type="fixed">
+    <!-- <joint name="chassis_joint" type="fixed">
         <parent link="base_link"/>
         <child link="chassis"/>
         <origin xyz="0 0 0.05"/>
-    </joint>
-    <link name="chassis">
+    </joint> -->
+    <link name="base_link">
         <!-- <xacro:insert_box_with_fillet size_x="0.28" size_y="0.2" size_z="${chassis_height}"
         fillet_radius="0.02" material="silver" x="0.09" y="0" z="${chassis_height/2}"/>
@@ -73,6 +73,6 @@
         </xacro:inertial_box>
     </link>
-    <gazebo reference="chassis">
-        <material>Gazebo/<color rgba="1.0 0.0 0.0 0.0"/>
+    <gazebo reference="base_link">
+        <material>Gazebo/<color rgba="0.25 0.25 0.25 1"/>
         </material>
     </gazebo>
@@ -80,5 +80,5 @@
     <!--  FRONT LEFT SERVO STEER LINK -->
     <joint name="front_left_servo_joint" type="revolute">
-        <parent link="chassis"/>
+        <parent link="base_link"/>
         <child link="front_left_servo"/>
         <origin xyz="${dist_btw_front_rear} 0.1 0"/>
@@ -126,5 +126,5 @@
     <!--  FRONT RIGHT SERVO STEER LINK -->
     <joint name="front_right_servo_joint" type="revolute">
-        <parent link="chassis"/>
+        <parent link="base_link"/>
         <child link="front_right_servo"/>
         <origin xyz="${dist_btw_front_rear} -0.1 0"/>
@@ -173,5 +173,5 @@
     <xacro:insert_drive_wheel
         base_name="rear_left_wheel"
-        parent_name="chassis"
+        parent_name="base_link"
         x="0" y="${wheel_seperation/2}" z="0"
         mass="${wheel_mass}"
@@ -189,5 +189,5 @@
     <xacro:insert_drive_wheel
         base_name="rear_right_wheel"
-        parent_name="chassis"
+        parent_name="base_link"
         x="0" y="${-wheel_seperation/2}" z="0"
         mass="${wheel_mass}"
@@ -205,5 +205,5 @@
     <xacro:insert_sonar
         base_name="sonar"
-        parent_name="chassis"
+        parent_name="base_link"
         x="${0.15+0.2+0.005}" y="0" z="${(chassis_height/2)}"
         mass="0.005"
@@ -214,5 +214,5 @@
     <xacro:insert_lidar
         base_name="lidar"
-        parent_name="chassis"
+        parent_name="base_link"
         x="0.2" y="0" z="${chassis_height+lidar_z_offset}"
         mass="0.05" samples="360"
@@ -223,5 +223,5 @@
     <!-- <xacro:insert_imu
         base_name="imu"
-        parent_name="chassis"
+        parent_name="base_link"
         x="0" y="0" z="${chassis_height}"/> -->
     <!--  normal camera style -->
@@ -230,5 +230,5 @@
     <xacro:insert_camera
         base_name="cam"
-        parent_name="chassis"
+        parent_name="base_link"
         x="0.15" y="0" z="${chassis_height+cam_z_offset+0.15}"
         mass="0.005"
